Commit message: Sync packages with the code deployed on the rover
Bring rover_driver and robot_description in line with the code running on the robot: the wheel-speed mix with its low-speed floor, the battery voltage topic, the Nav2 bringup launch file, the RF2O and Nav2 parameters, and the URDF laser yaw fix. Adds the ament_python package files missing from the previous layout.

File: src/robot_description/urdf/rover.urdf (robot description, URDF)
Before this commit: robot wave_rover, 2 links, 1 joints
Links:
- link base_link: geometry visual box size=0.250 0.227 0.100
Joints:
- joint base_to_laser: origin xyz=0.0 0.0 0.1685 rpy=0 0 0 -> xyz=0.0 0.0 0.1685 rpy=0 0 3.14159265
